Commit message: xhand-urdf

File: xhand_model/xhand_right_test.urdf (robot description, URDF)
Before this commit: robot xhand_right, 19 links, 18 joints
Joints:
- joint right_hand_index_bend_joint: axis 0 1 0 -> 0 -1 0; limit lower=-0.083 upper=0.297 effort=0.4 velocity=14.38 -> lower=-0.04 upper=0.297 effort=0.4 velocity=14.38
